Commit message: Add student exercise template with blanked parameters

File: src/rmitbot_description/urdf/common_properties.xacro (robot description, xacro)
@@ -2,4 +2,5 @@
 <robot name="rmitbot" xmlns:xacro="http://www.ros.org/wiki/xacro"
     xmlns:gz="http://gazebosim.org/schema">
+    <!-- ===================To be modified (optional but fun)============================ -->
     <!-- Color of the robot -->
     <material name="red">
@@ -27,4 +28,6 @@
         <color rgba="0.8 0.9 1.0 1.0" />
     </material>
+    <!-- ===================To be modified (optional but fun)============================ -->
+    <!-- ===================To be modified============================ -->
     <!-- Dimension of the robot -->
     <xacro:property name="base_mass" value="1.0" />
@@ -35,4 +38,5 @@
     <xacro:property name="wheel_radius" value="0.0425" />
     <xacro:property name="wheel_thickness" value="0.042" />
+    <!-- ===================To be modified============================ -->
     <!-- macro for calculating inertia -->
     <xacro:macro name="box_inertia" params="m x y z">

File: src/rmitbot_description/urdf/rmitbot_platform.xacro (robot description, xacro)
@@ -31,57 +31,15 @@
     </inertial>
   </link>
-  <!-- ======================================= -->
+  <!-- =================To be modified====================== -->
   <joint name="base_joint_2" type="fixed">
-    <parent link="base_link" />
-    <child link="base_link_2" />
-    <origin xyz="0 0 ${base_height}" rpy="0 0 0" />
   </joint>
-  <!-- ======================================= -->
+  <!-- =================To be modified====================== -->
   <link name="base_link_2">
-    <collision>
-      <origin xyz="0 0 0" rpy="0 0 0" />
-      <geometry>
-        <box size="${base_length} ${base_width} ${base_height}" />
-      </geometry>
-    </collision>
-    <visual>
-      <origin xyz="0 0 0" rpy="0 0 0" />
-      <geometry>
-        <box size="${base_length} ${base_width} ${base_height}" />
-      </geometry>
-      <material name="green" />
-    </visual>
-    <inertial>
-      <origin xyz="0 0 0" rpy="0 0 0" />
-      <mass value="${base_mass}" />
-      <xacro:box_inertia m="${base_mass}" x="${base_length}" y="${base_width}" z="${base_height}" />
-    </inertial>
   </link>
-  <!-- ======================================= -->
+  <!-- =================To be modified====================== -->
   <joint name="base_joint_3" type="fixed">
-    <parent link="base_link_2" />
-    <child link="base_link_3" />
-    <origin xyz="0 0 ${base_height}" rpy="0 0 0" />
   </joint>
-  <!-- ======================================= -->
+  <!-- =================To be modified====================== -->
   <link name="base_link_3">
-    <collision>
-      <origin xyz="0 0 0" rpy="0 0 0" />
-      <geometry>
-        <box size="${base_length} ${base_width} ${base_height}" />
-      </geometry>
-    </collision>
-    <visual>
-      <origin xyz="0 0 0" rpy="0 0 0" />
-      <geometry>
-        <box size="${base_length} ${base_width} ${base_height}" />
-      </geometry>
-      <material name="blue" />
-    </visual>
-    <inertial>
-      <origin xyz="0 0 0" rpy="0 0 0" />
-      <mass value="${base_mass}" />
-      <xacro:box_inertia m="${base_mass}" x="${base_length}" y="${base_width}" z="${base_height}" />
-    </inertial>
   </link>
 </robot>
